File: PID-simulator_kicad/PID-simulator_kicad.kicad_pcb (KiCad board)
At the start: 2 copper layers, 103.5 x 69.9 mm, 15 parts, among them SW1 Set, SW2 P, SW3 I, SW4 D, U1 L298N Module, U2 Motor, U3 GM009605 Screen, U4 6V In, U5 GY-521_MPU6050_v2

Commit message: schematics
Parts:
- added H3: MountingHole, MountingHole:MountingHole_3.2mm_M3, F.Cu at (188.7, 122.3)
Routing:
- net /D2 - IN1: track 92.8 -> 96.0 mm
- net GND: track 296.5 -> 294.4 mm
- added copper zone on B.Cu, net GND
- added copper zone on F.Cu, net GND
