File: PID-simulator_kicad/PID-simulator_kicad.kicad_sch (KiCad schematic)
At the start: 0 parts

Commit message: schematics and pcb
Parts:
- added A1: Arduino_Uno_R3_Shield, MyFootprints:Arduino_UNO_R3_shield_large, symbol PCM_arduino-library:Arduino_Uno_R3_Shield
- added R1, R2: 10k, Resistor_THT:R_Axial_DIN0207_L6.3mm_D2.5mm_P10.16mm_Horizontal, symbol Device:R
- added SW1: Set, MyFootprints:KY-040_rotary_encoder module_w_header_large, symbol My_Symbols:KY040_Rotary_Encoder_w_Switch
- added SW2: P, MyFootprints:KY-040_rotary_encoder module_w_header_large, symbol My_Symbols:KY040_Rotary_Encoder_w_Switch
- added SW3: I, MyFootprints:KY-040_rotary_encoder module_w_header_large, symbol My_Symbols:KY040_Rotary_Encoder_w_Switch
- added SW4: D, MyFootprints:KY-040_rotary_encoder module_w_header_large, symbol My_Symbols:KY040_Rotary_Encoder_w_Switch
- added U1: L298N Module, MyFootprints:MX1508 - L298N Dual H-Bridge Motor Driver Mini Module, symbol My_Symbols:L298N_Module
- added U2: Motor, MyFootprints:6-pin N20 DC Motor w Encoder, symbol My_Symbols:N20_DC_Motor_w_Encoder
- added U3: GM009605_0.96"_OLED_Screen, MyFootprints:SSD1306_I2C_0.96_OLED_display_large, symbol My_Symbols:GM009605_0.96{dblquote}_OLED_Screen
- added U4: 6V In, MyFootprints:2-pole_power_in_screw_terminal, symbol My_Symbols:2-pole_power_in_screw_terminal
Connections:
- new net +5V: A1.5V1 (5V), R1.1, R2.1, SW1.4 (VCC), SW2.4 (VCC), SW3.4 (VCC), SW4.4 (VCC), U2.5 (VCC), U3.2 (VDD)
- new net +6V: A1.VIN, U1.1 (+), U4.1 (+)
- new net D10: A1.D10 (D10_CS), SW3.1 (CLK)
- new net D11: A1.D11, SW3.2 (DT)
- new net D12: A1.D12, SW4.1 (CLK)
- new net D13: A1.D13, SW4.2 (DT)
- new net D2 - IN1: A1.D2 (D2_INT0), R2.2, U1.3 (IN1)
- new net D3 - IN2: A1.D3 (D3_INT1), R1.2, U1.4 (IN2)
- new net D4 - C1: A1.D4, U2.3 (C1)
- new net D5 - C2: A1.D5, U2.4 (C2)
- new net D6: A1.D6, SW1.1 (CLK)
- new net D7: A1.D7, SW1.2 (DT)
- new net D8: A1.D8, SW2.1 (CLK)
- new net D9: A1.D9, SW2.2 (DT)
- new net GND: A1.GND1 (GND), A1.GND2 (GND), A1.GND3 (GND), SW1.5 (GND), SW2.5 (GND), SW3.5 (GND), SW4.5 (GND), U1.2 (-), U2.2 (GND), U3.1 (GND), U4.2 (-)
- new net MotorA-1: U1.7 (MotorA-1), U2.1 (M1)
- new net MotorA-2: U1.8 (MotorA-2), U2.6 (M2)
- new net SCL: A1.SCL, U3.3 (SCK)
- new net SDA: A1.SDA, U3.4 (SDA)

Commit message: pcb update
Parts:
- added H1, H2: MountingHole, MountingHole:MountingHole_3.2mm_M3, symbol Mechanical:MountingHole
- added R3: 10k, Resistor_THT:R_Axial_DIN0207_L6.3mm_D2.5mm_P10.16mm_Horizontal, symbol Device:R
- added U5: GY-521_MPU6050_v2, MyFootprints:8-pin JST MPU6050, symbol My_Symbols:GY-521_MPU6050_v2
- A1: footprint MyFootprints:Arduino_UNO_R3_shield_large -> PCM_arduino-library:Arduino_Uno_R3_Shield
- U2: footprint MyFootprints:6-pin N20 DC Motor w Encoder -> MyFootprints:6-pin JST N20 DC Motor w Encoder
- U3: value GM009605_0.96"_OLED_Screen -> GM009605 Screen
Connections:
- net D4 - C1 is gone; now on net GND: A1.D4, U2.3 (C1)
- net +5V: now also U5.1 (VCC)
- net GND: now also R3.1, U5.2 (GND)
- net SCL: now also A1.A5, U5.3 (SCL); no longer A1.SCL
- net SDA: now also A1.A4, U5.4 (SDA); no longer A1.SDA
- net at A1.A0: now also R3.2, U5.7 (AD0)
- net D10 renamed D10 - I CLK
- net D11 renamed D11 - I DT
- net D12 renamed D12 - D CLK
- net D13 renamed D13 - D DT
- net D6 renamed D6 - Set CLK
- net D7 renamed D7 - Set DT
- net D8 renamed D8 - P CLK
- net D9 renamed D9 - P DT
Other:
- company: (none) -> Jonix
- title: (none) -> PID-Simulator
- moved on the sheet: R1, R2, SW1, SW2, SW3, SW4, U1, U2, U3, U4
